File: Hardware/Hardware.kicad_pcb (KiCad board)
At the start: 2 copper layers, 70 x 70 mm, 60 parts, among them J1 USB_C_Receptacle_USB2.0_16P, J2 Conn_01x02_Socket, J3 Conn_01x04_Pin, Q1 AO3400A, Q2 AO3401A, SW1 SW_Push, SW2 ON, SW3 SW_Push, U1 CH32V203CxTx, U2 AMS1117-3.3, U3 TP4056-42-ESOP8, U4 AMS1117-3.3

Commit message: feat: add donuts logo
Parts:
- added G***: LOGO, footprints:log_donuts, B.Cu at (85.0, 45.3)
